Commit message: feat:初步实现kuavo_s45的替换

File: humanoidverse/data/robots/biped_s45/urdf/biped_s45.urdf (robot description, URDF)
Before this commit: robot biped_s45, 47 links, 46 joints
Links:
- link base_link: geometry visual mesh filename=../meshes/torso.STL
- link camera: geometry visual mesh filename=../meshes/camera.STL
- link camera_base: geometry collision mesh filename=../meshes/camera_base.STL; visual mesh filename=../meshes/camera_base.STL
- link leg_l1_link: geometry visual mesh filename=../meshes/l_leg_roll.STL
- link leg_l2_link: geometry visual mesh filename=../meshes/l_leg_yaw.STL
- link leg_l3_link: geometry visual mesh filename=../meshes/l_leg_pitch.STL
- link leg_l4_link: geometry visual mesh filename=../meshes/l_knee.STL
- link leg_l5_link: geometry visual mesh filename=../meshes/l_foot_pitch.STL
- link leg_l6_link: geometry visual mesh filename=../meshes/l_foot_roll.STL
- link leg_r1_link: geometry visual mesh filename=../meshes/r_leg_roll.STL
- link leg_r2_link: geometry visual mesh filename=../meshes/r_leg_yaw.STL
- link leg_r3_link: geometry visual mesh filename=../meshes/r_leg_pitch.STL
- link leg_r4_link: geometry visual mesh filename=../meshes/r_knee.STL
- link leg_r5_link: geometry visual mesh filename=../meshes/r_foot_pitch.STL
- link leg_r6_link: geometry visual mesh filename=../meshes/r_foot_roll.STL
- link radar: geometry visual mesh filename=../meshes/radar.STL
- link zarm_l1_link: geometry visual mesh filename=../meshes/l_arm_pitch.STL
- link zarm_l2_link: geometry visual mesh filename=../meshes/l_arm_roll.STL
- link zarm_l3_link: geometry visual mesh filename=../meshes/l_arm_yaw.STL
- link zarm_l4_link: geometry visual mesh filename=../meshes/l_forearm.STL
- link zarm_l5_link: geometry visual mesh filename=../meshes/l_hand_yaw.STL
- link zarm_l6_link: geometry visual mesh filename=../meshes/l_hand_roll.STL
- link zarm_l7_link: geometry visual mesh filename=../meshes/l_hand_pitch.STL
- link zarm_r1_link: geometry visual mesh filename=../meshes/r_arm_pitch.STL
- link zarm_r2_link: geometry visual mesh filename=../meshes/r_arm_roll.STL
- link zarm_r3_link: geometry visual mesh filename=../meshes/r_arm_yaw.STL
- link zarm_r4_link: geometry visual mesh filename=../meshes/r_forearm.STL
- link zarm_r5_link: geometry visual mesh filename=../meshes/r_hand_yaw.STL
- link zarm_r6_link: geometry visual mesh filename=../meshes/r_hand_roll.STL
- link zarm_r7_link: geometry visual mesh filename=../meshes/r_hand_pitch.STL
- link zhead_1_link: geometry visual mesh filename=../meshes/head_yaw.STL
- link zhead_2_link: geometry visual mesh filename=../meshes/head_pitch.STL
